File: handle_bar/handle_barr/handle_barr.kicad_pcb (KiCad board)
At the start: 2 copper layers, 5 parts, among them J1 SPKR, U2 MCP73831-2-OT

Commit message: schematics completed
Parts:
- removed J1: SPKR, solderwirepad_1_02_SMD:SolderWirePad_1x02_SMD_5x5mm
- added C1: 10uf, Capacitor_THT:CP_Radial_D5.0mm_P2.00mm, B.Cu at (122.1, 44.9)
- added J2: MAX98357A 3V3, solderwirepad_1_02_SMD:SolderWirePad_1x07_SMD_1x3mm, B.Cu at (121.1, 64.4)
- added J3: PWR_SLIDE, solderwirepad_1_02_SMD:SolderWirePad_1x02_SMD_5x5mm, B.Cu at (112.7, 69.7)
- added J4: HRN_SW, solderwirepad_1_02_SMD:SolderWirePad_1x02_SMD_5x5mm, B.Cu at (137.9, 90.1)
- added J5: BAT, solderwirepad_1_02_SMD:SolderWirePad_1x02_SMD_5x5mm, B.Cu at (82.7, 68.8)
- added J6: PS2, solderwirepad_1_02_SMD:SolderWirePad_1x05_SMD_1x3mm, B.Cu at (96.7, 57.0)
- added J7: USB, solderwirepad_1_02_SMD:SolderWirePad_1x02_SMD_5x5mm, B.Cu at (125.3, 95.1)
- added R1: 2kΩ, Resistor_THT:R_Axial_DIN0207_L6.3mm_D2.5mm_P7.62mm_Horizontal, B.Cu at (148.4, 81.8)
- added U1: XIAO_ESP32C3, XIAO_ESP32C3:MODULE_XIAO_ESP32C3, F.Cu at (109.2, 54.3)
- U2: moved to B.Cu
- moved U2 28.8 mm to (97.1, 68.1), turned to 180 degrees
- moved D3 20.5 mm to (115.3, 94.4)
- moved D1 2.40 mm to (93.5, 94.5)

Commit message: routing_almost_done
Parts:
- added C2: 4.7, Capacitor_THT:C_Disc_D6.0mm_W2.5mm_P5.00mm, B.Cu at (90.6, 63.9)
- added C3: 4.7, Capacitor_THT:C_Disc_D6.0mm_W2.5mm_P5.00mm, B.Cu at (98.3, 66.3)
- added C4: 22uf, Capacitor_THT:CP_Radial_D5.0mm_P2.50mm, B.Cu at (94.6, 73.4)
- added PWR1: SW_SPST, solderwirepad_1_02_SMD:SolderWirePad_1x02_SMD_5x5mm, B.Cu at (124.4, 71.1)
- added R2: 220ko, Resistor_THT:R_Axial_DIN0207_L6.3mm_D2.5mm_P7.62mm_Horizontal, B.Cu at (125.7, 57.2)
- C1: footprint Capacitor_THT:CP_Radial_D5.0mm_P2.00mm -> Capacitor_THT:C_Disc_D7.5mm_W5.0mm_P5.00mm
- moved J3 68.4 mm to (93.9, 37.7), turned to 0 degrees
- moved R1 66.9 mm to (85.5, 59.4), turned to 0 degrees
- moved J6 60.6 mm to (89.0, 46.6), turned to -90 degrees
- moved D1 55.6 mm to (108.5, 41.0)
- moved J4 48.1 mm to (119.5, 37.8)
- moved D2 43.7 mm to (108.6, 50.9)
- moved D3 32.2 mm to (108.7, 62.9)
- moved J5 10.9 mm to (97.5, 46.1), turned to -90 degrees
- moved U2 6.30 mm to (96.9, 61.8)
- moved C1 3.82 mm to (125.9, 44.5)
- moved J3 2.53 mm to (110.3, 70.5)
- renumbered J4 to J3, J5 to J4, J6 to J5, J7 to J6
Connections:
- U1 pad 1: DIN -> unconnected-(U1-Pad1)
- U1 pad 10: unconnected-(U1-Pad10) -> BCLK
- U1 pad 11: unconnected-(U1-Pad11) -> LRCLK
- U1 pad 2: BCLK -> unconnected-(U1-Pad2)
- U1 pad 3: LRCLK -> unconnected-(U1-Pad3)
- U1 pad 4: unconnected-(U1-Pad4) -> VRx
- U1 pad 5: unconnected-(U1-Pad5) -> VRy
- U1 pad 6: unconnected-(U1-Pad6) -> SW_JS
- U1 pad 7: unconnected-(U1-Pad7) -> HORN
- U1 pad 8: unconnected-(U1-Pad8) -> DIN
- U2 pad 3: BAT_SYS -> BAT_RAW
Routing:
- net GND: track 0.00 -> 144.1 mm, vias 0 -> 2
- net 3V3: track 0.00 -> 84.6 mm, vias 0 -> 4
- net BAT_RAW: track 0.00 -> 84.3 mm
- net HORN: track 0.00 -> 25.0 mm, vias 0 -> 1
- net BAT_SYS: track 0.00 -> 25.0 mm
- net LED_DIN: track 0.00 -> 24.9 mm
- net VDD: track 0.00 -> 23.5 mm
- net LRCLK: track 0.00 -> 17.0 mm
- net BCLK: track 0.00 -> 13.1 mm
- net Net-(R1-Pad1): track 0.00 -> 11.8 mm
- net Net-(D2-Pad2): track 0.00 -> 10.8 mm
- net Net-(D1-Pad2): track 0.00 -> 8.68 mm
- net SD: track 0.00 -> 5.76 mm
- net VRy: track 0.00 -> 5.45 mm
- net SW_JS: track 0.00 -> 5.44 mm
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Other:
- board outline added: 48.5 x 48.6 mm

Commit message: done routing with edge
Parts:
- U1: moved to B.Cu
- turned U1 to 180 degrees
Connections:
- U1 pad 10: BCLK -> VRx
- U1 pad 11: LRCLK -> HORN
- U1 pad 2: unconnected-(U1-Pad2) -> LED_DIN
- U1 pad 4: VRx -> DIN
- U1 pad 5: VRy -> BCLK
- U1 pad 6: SW_JS -> LRCLK
- U1 pad 7: HORN -> unconnected-(U1-Pad7)
- U1 pad 8: DIN -> SW_JS
- U1 pad 9: LED_DIN -> VRy
Routing:
- net BAT_RAW: track 84.3 -> 72.4 mm
- net LED_DIN: track 24.9 -> 14.6 mm
- net GND: track 144.1 -> 151.9 mm, vias 2 -> 3
- net HORN: track 25.0 -> 17.9 mm, vias 1 -> 0
- net LRCLK: track 17.0 -> 10.7 mm
- net BCLK: track 13.1 -> 7.94 mm
- net SW_JS: track 5.44 -> 8.83 mm
- net 3V3: track 84.6 -> 87.9 mm
- net VRx: track 5.43 -> 8.48 mm
- net VRy: track 5.45 -> 8.41 mm
- net DIN: track 5.41 -> 7.12 mm
Other:
- outline, holes or cut-outs redrawn

Commit message: add joystick support on case
Parts:
- added GPS1: NEO6M, solderwirepad_1_02_SMD:SolderWirePad_1x04_SMD_1x3mm, F.Cu at (125.9, 39.9)
- renumbered R2 to R1, R1 to R2
Connections:
- U1 pad 3: unconnected-(U1-Pad3) -> SW_JS
- U1 pad 7: unconnected-(U1-Pad7) -> RX
- U1 pad 8: SW_JS -> TX
Routing:
- net TX: track 0.00 -> 49.8 mm, vias 0 -> 1
- net RX: track 0.00 -> 35.2 mm
- net SW_JS: track 8.83 -> 42.5 mm, vias 0 -> 1
- net GND: track 151.9 -> 160.4 mm, vias 3 -> 4
- net 3V3: track 87.9 -> 95.7 mm
Other:
- outline, holes or cut-outs redrawn

Commit message: ad poped display for indicator lights, made seprate pcb for daisy lights.
Parts:
- removed D1, D2, D3: WS2812B, LED_SMD:LED_WS2812B_PLCC4_5.0x5.0mm_P3.2mm
- added J3: Conn_01x03, solderwirepad_1_02_SMD:SolderWirePad_1x03_SMD_1x3mm, F.Cu at (108.7, 57.5)
- renumbered J3 to J4, J4 to J5, J5 to J6, J6 to J7
Routing:
- net 3V3: track 95.7 -> 51.0 mm, vias 4 -> 3
- net SW_JS: track 42.5 -> 29.7 mm, vias 1 -> 2
- net Net-(D2-Pad2): track 10.8 -> 0.00 mm
- net GND: track 160.4 -> 150.4 mm, vias 4 -> 3
- net Net-(D1-Pad2): track 8.68 -> 0.00 mm
- net BAT_RAW: track 72.4 -> 70.0 mm
Other:
- outline, holes or cut-outs redrawn
