File: handle_bar/handle_barr/handle_barr.kicad_sch (KiCad schematic)
At the start: 14 parts, among them J1 SPKR, J2 MAX98357A 3V3, J3 PWR_SLIDE, J4 HRN_SW, J5 BAT, J6 PS2, J7 USB, U1 XIAO_ESP32C3, U2 MCP73831-2-OT

Commit message: schematics completed
Parts:
- removed J3: PWR_SLIDE, symbol Connector_Generic:Conn_01x02
- added C2, C3: 4.7, Capacitor_SMD:C_0805_2012Metric_Pad1.18x1.45mm_HandSolder, symbol Device:C
- added PWR1: SW_SPST, solderwirepad_1_02_SMD:SolderWirePad_1x02_SMD_5x5mm, symbol Switch:SW_SPST
- added R2: 220ko, Resistor_THT:R_Axial_DIN0207_L6.3mm_D2.5mm_P7.62mm_Horizontal, symbol Device:R
- C1: footprint (none) -> Capacitor_THT:CP_Radial_D5.0mm_P2.00mm
- J1: footprint solderwirepad_1_02_SMD:SolderWirePad_1x02_SMD_5x5mm -> (none)
- J2: footprint (none) -> solderwirepad_1_02_SMD:SolderWirePad_1x07_SMD_1x3mm
- J3: renamed from J4; footprint (none) -> solderwirepad_1_02_SMD:SolderWirePad_1x02_SMD_5x5mm
- J4: renamed from J5; footprint (none) -> solderwirepad_1_02_SMD:SolderWirePad_1x02_SMD_5x5mm
- J5: renamed from J6; footprint (none) -> solderwirepad_1_02_SMD:SolderWirePad_1x05_SMD_1x3mm
- J6: renamed from J7; footprint (none) -> solderwirepad_1_02_SMD:SolderWirePad_1x02_SMD_5x5mm
- R1: footprint (none) -> Resistor_THT:R_Axial_DIN0207_L6.3mm_D2.5mm_P7.62mm_Horizontal
Connections:
- net +3.3V: now also R2.2
- net BAT_RAW: now also U2.3 (VBAT), C3.2, PWR1.2 (B)
- net BAT_SYS: now also PWR1.1 (A); no longer U2.3 (VBAT)
- net GND: now also J6.2 (Pin_2), C2.2, C3.1; no longer J6.4 (Pin_4)
- net SD: now also R2.1
- net SW_JS: now also U1.6 (D5)
- net VDD: now also C2.1
- net VRx: now also U1.4 (D3)
- net VRy: now also U1.5 (D4)

Commit message: routing_almost_done
Parts:
- added C4: 22uf, Capacitor_THT:CP_Radial_D5.0mm_P2.50mm, symbol Device:C
- C1: footprint Capacitor_THT:CP_Radial_D5.0mm_P2.00mm -> Capacitor_THT:C_Disc_D7.5mm_W5.0mm_P5.00mm
- C2, C3: footprint Capacitor_SMD:C_0805_2012Metric_Pad1.18x1.45mm_HandSolder -> Capacitor_THT:C_Disc_D6.0mm_W2.5mm_P5.00mm
Connections:
- net BAT_SYS: now also C4.1
- net BCLK: now also U1.10 (D9); no longer U1.2 (D1)
- net GND: now also C4.2
- net HORN: now also U1.7 (TX_D6)
- net LRCLK: now also U1.11 (D10); no longer U1.3 (D2)
Changed lines of the file:
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@@
+    (stroke (width 0) (type default) (color 0 0 0 0))
+  )
+  (wire (pts (xy 195.58 90.17) (xy 203.2 90.17))
     (stroke (width 0) (type default) (color 0 0 0 0))
   )
@@
     (stroke (width 0) (type default) (color 0 0 0 0))
   )
+  (wire (pts (xy 196.85 82.55) (xy 203.2 82.55))
+    (stroke (width 0) (type default) (color 0 0 0 0))
+  )
   (wire (pts (xy 128.27 68.58) (xy 134.62 68.58))
     (stroke (width 0) (type default) (color 0 0 0 0))
@@
     )
   )
-  (global_label "BCLK" (shape input) (at 43.18 48.26 180) (fields_autoplaced)
-    (effects (font (size 1 1)) (justify right))
-    (property "Intersheet References" "${INTERSHEET_REFS}" (id 0) (at 37.4705 48.1975 0)
-      (effects (font (size 1 1)) (justify right) hide)
-    )
-  )
   (global_label "GND" (shape input) (at 149.86 102.87 270) (fields_autoplaced)
     (effects (font (size 1 1)) (justify right))
     (property "Intersheet References" "${INTERSHEET_REFS}" (id 0) (at 149.7975 107.8176 90)
+      (effects (font (size 1 1)) (justify right) hide)
+    )
+  )
+  (global_label "BCLK" (shape input) (at 78.74 53.34 0) (fields_autoplaced)
+    (effects (font (size 1 1)) (justify left))
+    (property "Intersheet References" "${INTERSHEET_REFS}" (id 0) (at 84.4495 53.4025 0)
+      (effects (font (size 1 1)) (justify left) hide)
+    )
+  )
+  (global_label "BAT_SYS" (shape input) (at 196.85 82.55 180) (fields_autoplaced)
+    (effects (font (size 1 1)) (justify right))
+    (property "Intersheet References" "${INTERSHEET_REFS}" (id 0) (at 188.8071 82.6125 0)
       (effects (font (size 1 1)) (justify right) hide)
     )
@@
     )
   )
+  (global_label "LRCLK" (shape input) (at 78.74 55.88 0) (fields_autoplaced)
+    (effects (font (size 1 1)) (justify left))
+    (property "Intersheet References" "${INTERSHEET_REFS}" (id 0) (at 85.259 55.9425 0)
+      (effects (font (size 1 1)) (justify left) hide)
+    )
+  )
+  (global_label "HORN" (shape input) (at 78.74 45.72 0) (fields_autoplaced)
+    (effects (font (size 1 1)) (justify left))
+    (property "Intersheet References" "${INTERSHEET_REFS}" (id 0) (at 84.7829 45.7825 0)
+      (effects (font (size 1 1)) (justify left) hide)
+    )
+  )
   (global_label "GND" (shape input) (at 161.29 50.8 270) (fields_autoplaced)
     (effects (font (size 1 1)) (justify right))
@@
     (property "Intersheet References" "${INTERSHEET_REFS}" (id 0) (at 83.6876 63.5625 0)
       (effects (font (size 1 1)) (justify left) hide)
+    )
+  )
+  (global_label "GND" (shape input) (at 195.58 90.17 180) (fields_autoplaced)
+    (effects (font (size 1 1)) (justify right))
+    (property "Intersheet References" "${INTERSHEET_REFS}" (id 0) (at 190.6324 90.1075 0)
+      (effects (font (size 1 1)) (justify right) hide)
     )
   )
@@
     )
   )
-  (global_label "LRCLK" (shape input) (at 43.18 50.8 180) (fields_autoplaced)
-    (effects (font (size 1 1)) (justify right))
-    (property "Intersheet References" "${INTERSHEET_REFS}" (id 0) (at 36.661 50.7375 0)
-      (effects (font (size 1 1)) (justify right) hide)
-    )
-  )
   (global_label "VRy" (shape input) (at 43.18 55.88 180) (fields_autoplaced)
     (effects (font (size 1 1)) (justify right))
@@
       (effects (font (size 1.27 1.27)) (justify left))
     )
-    (property "Footprint" "Capacitor_THT:CP_Radial_D5.0mm_P2.00mm" (id 2) (at 129.2352 76.2 0)
+    (property "Footprint" "Capacitor_THT:C_Disc_D7.5mm_W5.0mm_P5.00mm" (id 2) (at 129.2352 76.2 0)
       (effects (font (size 1.27 1.27)) hide)
     )
@@
     )
     (property "Datasheet" "~" (id 3) (at 189.23 41.91 0)
+      (effects (font (size 1.27 1.27)) hide)
+    )
+    (pin "1")
+    (pin "2")
+  )
+  (symbol (lib_id "Device:C") (at 203.2 86.36 0) (unit 1)
+    (in_bom yes) (on_board yes) (fields_autoplaced)
+    (property "Reference" "C4" (id 0) (at 207.01 85.0899 0)
+      (effects (font (size 1.27 1.27)) (justify left))
+    )
+    (property "Value" "22uf" (id 1) (at 207.01 87.6299 0)
+      (effects (font (size 1.27 1.27)) (justify left))
+    )
+    (property "Footprint" "Capacitor_THT:CP_Radial_D5.0mm_P2.50mm" (id 2) (at 204.1652 90.17 0)
+      (effects (font (size 1.27 1.27)) hide)
+    )
+    (property "Datasheet" "~" (id 3) (at 203.2 86.36 0)
       (effects (font (size 1.27 1.27)) hide)
     )
@@
     (property "Reference" "C2" (id 0) (at 170.18 68.58 90))
     (property "Value" "4.7" (id 1) (at 170.18 71.12 90))
-    (property "Footprint" "Capacitor_SMD:C_0805_2012Metric_Pad1.18x1.45mm_HandSolder" (id 2) (at 173.99 75.2348 0)
+    (property "Footprint" "Capacitor_THT:C_Disc_D6.0mm_W2.5mm_P5.00mm" (id 2) (at 173.99 75.2348 0)
       (effects (font (size 1.27 1.27)) hide)
     )
@@
       (effects (font (size 1.27 1.27)) (justify right))
     )
-    (property "Footprint" "Capacitor_SMD:C_0805_2012Metric_Pad1.18x1.45mm_HandSolder" (id 2) (at 173.0248 91.44 0)
+    (property "Footprint" "Capacitor_THT:C_Disc_D6.0mm_W2.5mm_P5.00mm" (id 2) (at 173.0248 91.44 0)
       (effects (font (size 1.27 1.27)) hide)
     )
@@
     )
     (path "/07e0a7f3-471a-48bc-9358-26b2e08f3961"
-      (reference "C1") (unit 1) (value "10uf") (footprint "Capacitor_THT:CP_Radial_D5.0mm_P2.00mm")
+      (reference "C1") (unit 1) (value "10uf") (footprint "Capacitor_THT:C_Disc_D7.5mm_W5.0mm_P5.00mm")
     )
     (path "/774afdf2-62a0-447f-bed5-136f0c5054a8"
-      (reference "C2") (unit 1) (value "4.7") (footprint "Capacitor_SMD:C_0805_2012Metric_Pad1.18x1.45mm_HandSolder")
+      (reference "C2") (unit 1) (value "4.7") (footprint "Capacitor_THT:C_Disc_D6.0mm_W2.5mm_P5.00mm")
     )
     (path "/9c00dbf8-5517-42b9-b038-8357a3da1e8a"
-      (reference "C3") (unit 1) (value "4.7") (footprint "Capacitor_SMD:C_0805_2012Metric_Pad1.18x1.45mm_HandSolder")
+      (reference "C3") (unit 1) (value "4.7") (footprint "Capacitor_THT:C_Disc_D6.0mm_W2.5mm_P5.00mm")
+    )
+    (path "/2e4f2f23-8979-495a-ac06-bbe38d80e056"
+      (reference "C4") (unit 1) (value "22uf") (footprint "Capacitor_THT:CP_Radial_D5.0mm_P2.50mm")
     )
     (path "/18019663-0f9f-4d73-bdf5-b9981c3a9216"

Commit message: done routing with edge
Connections:
- net BCLK: now also U1.5 (D4); no longer U1.10 (D9)
- net DIN: no longer U1.1 (D0)
- net LED_DIN: now also U1.4 (D3); no longer U1.9 (D8)
- net LRCLK: now also U1.6 (D5); no longer U1.11 (D10)
- net SW_JS: now also U1.8 (RX_D7); no longer U1.6 (D5)
- net VRx: now also U1.9 (D8); no longer U1.4 (D3)
- net VRy: now also U1.10 (D9); no longer U1.5 (D4)
Changed lines of the file:
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@@
+    )
+  )
+  (global_label "VRy" (shape input) (at 78.74 53.34 0) (fields_autoplaced)
+    (effects (font (size 1 1)) (justify left))
+    (property "Intersheet References" "${INTERSHEET_REFS}" (id 0) (at 83.259 53.2775 0)
+      (effects (font (size 1 1)) (justify left) hide)
     )
   )
@@
     )
   )
+  (global_label "SW_JS" (shape input) (at 78.74 48.26 0) (fields_autoplaced)
+    (effects (font (size 1 1)) (justify left))
+    (property "Intersheet References" "${INTERSHEET_REFS}" (id 0) (at 85.2114 48.3225 0)
+      (effects (font (size 1 1)) (justify left) hide)
+    )
+  )
   (global_label "3V3" (shape input) (at 161.29 35.56 90) (fields_autoplaced)
     (effects (font (size 1 1)) (justify left))
@@
     (property "Intersheet References" "${INTERSHEET_REFS}" (id 0) (at 149.7975 107.8176 90)
       (effects (font (size 1 1)) (justify right) hide)
-    )
-  )
-  (global_label "BCLK" (shape input) (at 78.74 53.34 0) (fields_autoplaced)
-    (effects (font (size 1 1)) (justify left))
-    (property "Intersheet References" "${INTERSHEET_REFS}" (id 0) (at 84.4495 53.4025 0)
-      (effects (font (size 1 1)) (justify left) hide)
     )
   )
@@
     )
   )
+  (global_label "LRCLK" (shape input) (at 43.18 58.42 180) (fields_autoplaced)
+    (effects (font (size 1 1)) (justify right))
+    (property "Intersheet References" "${INTERSHEET_REFS}" (id 0) (at 36.661 58.3575 0)
+      (effects (font (size 1 1)) (justify right) hide)
+    )
+  )
   (global_label "LED_DIN" (shape input) (at 104.14 43.18 180) (fields_autoplaced)
     (effects (font (size 1 1)) (justify right))
@@
     )
   )
-  (global_label "VRx" (shape input) (at 43.18 53.34 180) (fields_autoplaced)
-    (effects (font (size 1 1)) (justify right))
-    (property "Intersheet References" "${INTERSHEET_REFS}" (id 0) (at 38.6133 53.2775 0)
-      (effects (font (size 1 1)) (justify right) hide)
-    )
-  )
   (global_label "3V3" (shape input) (at 78.74 38.1 0) (fields_autoplaced)
     (effects (font (size 1 1)) (justify left))
@@
     )
   )
-  (global_label "SW_JS" (shape input) (at 43.18 58.42 180) (fields_autoplaced)
-    (effects (font (size 1 1)) (justify right))
-    (property "Intersheet References" "${INTERSHEET_REFS}" (id 0) (at 36.7086 58.3575 0)
-      (effects (font (size 1 1)) (justify right) hide)
+  (global_label "VRx" (shape input) (at 78.74 50.8 0) (fields_autoplaced)
+    (effects (font (size 1 1)) (justify left))
+    (property "Intersheet References" "${INTERSHEET_REFS}" (id 0) (at 83.3067 50.8625 0)
+      (effects (font (size 1 1)) (justify left) hide)
     )
   )
@@
     )
   )
-  (global_label "LRCLK" (shape input) (at 78.74 55.88 0) (fields_autoplaced)
-    (effects (font (size 1 1)) (justify left))
-    (property "Intersheet References" "${INTERSHEET_REFS}" (id 0) (at 85.259 55.9425 0)
-      (effects (font (size 1 1)) (justify left) hide)
-    )
-  )
   (global_label "HORN" (shape input) (at 78.74 45.72 0) (fields_autoplaced)
     (effects (font (size 1 1)) (justify left))
@@
     )
   )
+  (global_label "BCLK" (shape input) (at 43.18 55.88 180) (fields_autoplaced)
+    (effects (font (size 1 1)) (justify right))
+    (property "Intersheet References" "${INTERSHEET_REFS}" (id 0) (at 37.4705 55.8175 0)
+      (effects (font (size 1 1)) (justify right) hide)
+    )
+  )
   (global_label "GND" (shape input) (at 195.58 90.17 180) (fields_autoplaced)
     (effects (font (size 1 1)) (justify right))
@@
     )
   )
-  (global_label "DIN" (shape input) (at 43.18 45.72 180) (fields_autoplaced)
-    (effects (font (size 1 1)) (justify right))
-    (property "Intersheet References" "${INTERSHEET_REFS}" (id 0) (at 38.7562 45.6575 0)
-      (effects (font (size 1 1)) (justify right) hide)
-    )
-  )
   (global_label "GND" (shape input) (at 184.15 44.45 180) (fields_autoplaced)
     (effects (font (size 1 1)) (justify right))
@@
     )
   )
-  (global_label "LED_DIN" (shape input) (at 78.74 50.8 0) (fields_autoplaced)
-    (effects (font (size 1 1)) (justify left))
-    (property "Intersheet References" "${INTERSHEET_REFS}" (id 0) (at 86.64 50.8625 0)
-      (effects (font (size 1 1)) (justify left) hide)
-    )
-  )
   (global_label "VRx" (shape input) (at 215.9 44.45 180) (fields_autoplaced)
     (effects (font (size 1 1)) (justify right))
@@
     (effects (font (size 1 1)) (justify right))
     (property "Intersheet References" "${INTERSHEET_REFS}" (id 0) (at 211.2381 41.8475 0)
+      (effects (font (size 1 1)) (justify right) hide)
+    )
+  )
+  (global_label "DIN" (shape input) (at 31.75 48.26 180) (fields_autoplaced)
+    (effects (font (size 1 1)) (justify right))
+    (property "Intersheet References" "${INTERSHEET_REFS}" (id 0) (at 27.3262 48.1975 0)
       (effects (font (size 1 1)) (justify right) hide)
     )
@@
     )
   )
-  (global_label "VRy" (shape input) (at 43.18 55.88 180) (fields_autoplaced)
-    (effects (font (size 1 1)) (justify right))
-    (property "Intersheet References" "${INTERSHEET_REFS}" (id 0) (at 38.661 55.8175 0)
-      (effects (font (size 1 1)) (justify right) hide)
-    )
-  )
   (global_label "GND" (shape input) (at 173.99 76.2 0) (fields_autoplaced)
     (effects (font (size 1 1)) (justify left))
@@
     )
   )
+  (global_label "LED_DIN" (shape input) (at 43.18 53.34 180) (fields_autoplaced)
+    (effects (font (size 1 1)) (justify right))
+    (property "Intersheet References" "${INTERSHEET_REFS}" (id 0) (at 35.28 53.2775 0)
+      (effects (font (size 1 1)) (justify right) hide)
+    )
+  )

Commit message: started_handle_bar_assembly
Connections:
- net DIN: now also U1.4 (D3)
- net HORN: now also U1.11 (D10); no longer U1.7 (TX_D6)
- net LED_DIN: now also U1.2 (D1); no longer U1.4 (D3)
- net VRx: now also U1.10 (D9); no longer U1.9 (D8)
- net VRy: now also U1.9 (D8); no longer U1.10 (D9)
Changed lines of the file:
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@@
+    )
+  )
+  (global_label "LED_DIN" (shape input) (at 43.18 48.26 180) (fields_autoplaced)
+    (effects (font (size 1 1)) (justify right))
+    (property "Intersheet References" "${INTERSHEET_REFS}" (id 0) (at 35.28 48.1975 0)
+      (effects (font (size 1 1)) (justify right) hide)
     )
   )
@@
     (property "Intersheet References" "${INTERSHEET_REFS}" (id 0) (at 124.3975 69.4319 90)
       (effects (font (size 1 1)) (justify right) hide)
-    )
-  )
-  (global_label "VRy" (shape input) (at 78.74 53.34 0) (fields_autoplaced)
-    (effects (font (size 1 1)) (justify left))
-    (property "Intersheet References" "${INTERSHEET_REFS}" (id 0) (at 83.259 53.2775 0)
-      (effects (font (size 1 1)) (justify left) hide)
     )
   )
@@
     )
   )
+  (global_label "HORN" (shape input) (at 78.74 55.88 0) (fields_autoplaced)
+    (effects (font (size 1 1)) (justify left))
+    (property "Intersheet References" "${INTERSHEET_REFS}" (id 0) (at 84.7829 55.9425 0)
+      (effects (font (size 1 1)) (justify left) hide)
+    )
+  )
   (global_label "DIN" (shape input) (at 137.16 62.23 180) (fields_autoplaced)
     (effects (font (size 1 1)) (justify right))
@@
     )
   )
-  (global_label "VRx" (shape input) (at 78.74 50.8 0) (fields_autoplaced)
-    (effects (font (size 1 1)) (justify left))
-    (property "Intersheet References" "${INTERSHEET_REFS}" (id 0) (at 83.3067 50.8625 0)
-      (effects (font (size 1 1)) (justify left) hide)
+  (global_label "DIN" (shape input) (at 43.18 53.34 180) (fields_autoplaced)
+    (effects (font (size 1 1)) (justify right))
+    (property "Intersheet References" "${INTERSHEET_REFS}" (id 0) (at 38.7562 53.2775 0)
+      (effects (font (size 1 1)) (justify right) hide)
     )
   )
@@
     )
   )
-  (global_label "HORN" (shape input) (at 78.74 45.72 0) (fields_autoplaced)
-    (effects (font (size 1 1)) (justify left))
-    (property "Intersheet References" "${INTERSHEET_REFS}" (id 0) (at 84.7829 45.7825 0)
-      (effects (font (size 1 1)) (justify left) hide)
-    )
-  )
   (global_label "GND" (shape input) (at 161.29 50.8 270) (fields_autoplaced)
     (effects (font (size 1 1)) (justify right))
@@
     )
   )
+  (global_label "VRx" (shape input) (at 78.74 53.34 0) (fields_autoplaced)
+    (effects (font (size 1 1)) (justify left))
+    (property "Intersheet References" "${INTERSHEET_REFS}" (id 0) (at 83.3067 53.4025 0)
+      (effects (font (size 1 1)) (justify left) hide)
+    )
+  )
   (global_label "BCLK" (shape input) (at 43.18 55.88 180) (fields_autoplaced)
     (effects (font (size 1 1)) (justify right))
@@
     (effects (font (size 1 1)) (justify right))
     (property "Intersheet References" "${INTERSHEET_REFS}" (id 0) (at 211.2381 41.8475 0)
-      (effects (font (size 1 1)) (justify right) hide)
-    )
-  )
-  (global_label "DIN" (shape input) (at 31.75 48.26 180) (fields_autoplaced)
-    (effects (font (size 1 1)) (justify right))
-    (property "Intersheet References" "${INTERSHEET_REFS}" (id 0) (at 27.3262 48.1975 0)
       (effects (font (size 1 1)) (justify right) hide)
     )
@@
     )
   )
+  (global_label "VRy" (shape input) (at 78.74 50.8 0) (fields_autoplaced)
+    (effects (font (size 1 1)) (justify left))
+    (property "Intersheet References" "${INTERSHEET_REFS}" (id 0) (at 83.259 50.7375 0)
+      (effects (font (size 1 1)) (justify left) hide)
+    )
+  )
   (global_label "GND" (shape input) (at 215.9 39.37 180) (fields_autoplaced)
     (effects (font (size 1 1)) (justify right))
@@
     )
   )
-  (global_label "LED_DIN" (shape input) (at 43.18 53.34 180) (fields_autoplaced)
-    (effects (font (size 1 1)) (justify right))
-    (property "Intersheet References" "${INTERSHEET_REFS}" (id 0) (at 35.28 53.2775 0)
-      (effects (font (size 1 1)) (justify right) hide)
-    )
-  )
